File: hardware/gbikePCB.sch (EAGLE design)
At the start: 19 parts, among them Q1 16M, U1 nRF51822

Commit message: updated pcb file
Parts:
- removed JP3, JP4: (no value), AUSER KJ:M07
- removed Q1: 16M, APM_v2:DIYDRONES3_RESONATORSMD
- removed U$2: ANTENNA_INVERTED_F_ANTENNA-3, nRF51822:ANTENNA_INVERTED_F_ANTENNA-3
- added ANT1: AN2051, Tiny_BLE_V1.0:CONNECTOR_ANTENNA-2.4GHZ-0.5DBIAN2051
- added C1, C12: 100nF, Tiny_BLE_V1.0:DISCRETE_C-0603
- added C13: 2.2nF, Tiny_BLE_V1.0:DISCRETE_C-0603
- added C2: 0.1uF, Tiny_BLE_V1.0:DISCRETE_C-0603
- added D1: led1, Tiny_BLE_V1.0:DISCRETE_LED0603
- added NRF51822: nRF51822, nRF51822ModifiedFortValue:NRF51822_NRF51822_NRF51822
- added Q2: 16M, APM_v2:DIYDRONES3_RESONATORSMD
- added R1: 4.7K, Tiny_BLE_V1.0:DISCRETE_R-0603
- added R4, R5: 10k, Tiny_BLE_V1.0:DISCRETE_R-0603
- C10, C11, C3, C4, C5, C6, C7, C8, C9: device SparkFun:CAP0603-CAP -> Tiny_BLE_V1.0:DISCRETE_C-0603
- JP1: value (none) -> Interface; device AUSER KJ:M07 -> pinhead:PINHD-1X6
- JP2: value (none) -> SWD; device AUSER KJ:M07 -> pinhead:PINHD-1X4
- L1, L2, L3: device AUSER KJ:L0603 -> Tiny_BLE_V1.0:DISCRETE_L0603
- U1: value nRF51822 -> mpu6050; device nRF51822:NRF51822_NRF51822MYTEST -> nRF51822:TINY_BLE_V1.0_TEMPLATE_MPU-6050???¡¥
Connections:
- removed net N$1: Q1.3, U1.XC2
- removed net N$14: JP1.1, JP3.1, U1.P0.03
- removed net N$15: JP2.7, JP4.7, U1.P0.04
- removed net N$16: JP2.6, JP4.6, U1.P0.05
- new net IMU_INT: NRF51822.P0.29, U1.INT
- new net N$18: C12.1, U1.REGOUT
- new net N$19: C13.1, U1.CPOUT
- new net P04: D1.+, NRF51822.P0.04
- new net SCL: NRF51822.P0.28, R5.2, U1.SCL
- new net SDA: NRF51822.P0.27, R4.2, U1.SDA
- net N$10: now also JP1.2, NRF51822.P0.01; no longer JP1.4, JP3.4, U1.P0.00
- net N$11: now also NRF51822.P0.02; no longer JP3.3, U1.P0.01
- net N$12: now also NRF51822.ANT1; no longer U1.ANT1
- net N$13: now also JP1.4, NRF51822.P0.03; no longer JP1.2, JP3.2, U1.P0.02
- net N$17: now also D1.-, R1.1; no longer JP2.5, JP4.5, U1.P0.06
- net N$2: now also JP1.1, NRF51822.P0.00; no longer Q1.1, U1.XC1
- net N$28: now also NRF51822.SWDIO/NRESET; no longer JP4.3, U1.SWDIO/NRESET
- net N$29: now also NRF51822.SWDCLK; no longer JP4.2, U1.SWDCLK
- net N$3: now also NRF51822.VDD_PA; no longer U1.VDD_PA
- net N$4: now also NRF51822.XC2, Q2.3; no longer JP1.7, JP3.7, U1.P0.26
- net N$5: now also NRF51822.DEC1; no longer U1.DEC1
- net N$6: now also NRF51822.ANT2; no longer U1.ANT2
- net N$8: now also ANT1.1; no longer U$2.FEED
- net N$9: now also NRF51822.XC1, Q2.1; no longer JP1.6, JP3.6, U1.P0.27
- net VDD: now also C1.1, C2.2, JP1.6, JP2.4, NRF51822.AVDD, NRF51822.AVDD_2, NRF51822.DEC2, NRF51822.VDD, NRF51822.VDD_2, R1.2, R4.1, R5.1, U1.VLOGIC; no longer JP1.5, JP3.5, U1.AVDD, U1.AVDD_2, U1.DEC2, U1.VDD_2
- net VSS: now also C1.2, C12.2, C13.2, C2.1, JP1.5, NRF51822.BASE, NRF51822.VSS, NRF51822.VSS_2, NRF51822.VSS_3, Q2.2, U1.AD0, U1.CLKIN, U1.FSYNC, U1.GND; no longer JP2.4, JP4.1, JP4.4, Q1.2, U$2.GND, U$2.GND@1, U1.BASE, U1.VSS, U1.VSS_2, U1.VSS_3
Other:
- note added: "Blue Magic v0.1 Shanghai Geek Center"
